File: test_spc500.kicad_sch (KiCad schematic)
At the start: 0 parts

Commit message: update info
Other:
- company: (none) -> @stoppattern
- title: (none) -> test_scp500
Changed lines of the file:
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@@
 	(generator_version "10.0")
 	(paper "A4")
+	(title_block
+		(title "test_scp500")
+		(date "2026-09-08")
+		(rev "0.01")
+		(company "@stoppattern")
+		(comment 1 "SPC500 テスト基板")
+	)
 	(sheet_instances
 		(path "/"

Commit message: paste sch
Parts:
- added C10, C11, C12, C13, C14, C15, C16, C17, C18, C20, C21, C22, C6, C7, C8: 100n, Capacitor_SMD:C_0402_1005Metric, symbol Device:C
- added C19: 2.2u, Capacitor_SMD:C_0603_1608Metric, symbol Device:C
- added C5, C9: 15p, Capacitor_SMD:C_0603_1608Metric, symbol Device:C
- added H1, H2, H3, H4: MountingHole, MountingHole:MountingHole_3.2mm_M3, symbol Mechanical:MountingHole
- added J3: SWD, Connector_PinHeader_2.54mm:PinHeader_1x03_P2.54mm_Vertical, symbol Connector_Generic:Conn_01x03
- added LD1: ERR, LED_SMD:LED_0603_1608Metric, symbol Device:LED
- added LD2: TX, LED_SMD:LED_0603_1608Metric, symbol Device:LED
- added LD3: LED, LED_SMD:LED_0603_1608Metric, symbol Device:LED
- added Q5, Q6, Q7: AO3400A, Package_TO_SOT_SMD:SOT-23, symbol Transistor_FET:AO3400A
- added R13, R15, R19, R20, R22, R24, R26: 1k, Resistor_SMD:R_0603_1608Metric, symbol Device:R
- added R14: 0, Resistor_SMD:R_0603_1608Metric, symbol Device:R
- added R16, R17, R18: 22, Resistor_SMD:R_0603_1608Metric, symbol Device:R
- added R21, R23, R25: 10k, Resistor_SMD:R_0603_1608Metric, symbol Device:R
- added SW1: RUN, Button_Switch_SMD:SW_Push_SPST_NO_Alps_SKRK, symbol Switch:SW_Push
- added SW2: BOOTSEL, Button_Switch_SMD:SW_Push_SPST_NO_Alps_SKRK, symbol Switch:SW_Push
- added SW3: SW, Button_Switch_SMD:SW_Push_SPST_NO_Alps_SKRK, symbol Switch:SW_Push
- added U11: RP2354A, Package_DFN_QFN:QFN-60-1EP_7x7mm_P0.4mm_EP3.4x3.4mm, symbol MCU_RaspberryPi:RP2354A
- added Y1: 12MHz, Crystal:Crystal_SMD_3225-4Pin_3.2x2.5mm, symbol Device:Crystal_GND24
Connections:
- new net: LD2.2 (A), R24.1
- new net: LD1.2 (A), R22.1
- new net: LD3.1 (K), Q7.3 (D)
- new net: LD3.2 (A), R26.1
- new net: LD1.1 (K), Q5.3 (D)
- new net: LD2.1 (K), Q6.3 (D)
- new net: C5.1, R14.1, Y1.1
- new net: C9.1, R15.1, Y1.3
- new net: C19.1, C21.1, R18.1, U11.44 (ADC_AVDD)
- new net: C10.1, R13.1, SW1.2
- new net: C18.1, R19.1, SW2.2
- new net +1V1: C16.1, C17.1, C20.1, U11.23 (DVDD), U11.39 (DVDD), U11.6 (DVDD)
- new net +3V3: C11.1, C12.1, C13.1, C14.1, C15.1, C22.1, C6.1, C7.1, C8.1, R18.2, R21.2, R22.2, R24.2, R26.2, SW3.1, U11.1 (IOVDD), U11.11 (IOVDD), U11.20 (IOVDD), U11.30 (IOVDD), U11.38 (IOVDD), U11.45 (IOVDD), U11.46 (VREG_AVDD), U11.49 (VREG_VIN), U11.53 (USB_OTP_VDD), U11.54 (QSPI_IOVDD)
- new net D+: R17.2, U11.52 (USB_DP)
- new net D-: R16.2, U11.51 (USB_DM)
- new net Err: Q5.1 (G), R21.1, U11.3 (GPIO1)
- new net GND: C10.2, C11.2, C12.2, C13.2, C14.2, C15.2, C16.2, C17.2, C18.2, C19.2, C20.2, C21.2, C5.2, C6.2, C7.2, C8.2, C9.2, J3.2 (Pin_2), Q5.2 (S), Q6.2 (S), Q7.2 (S), R20.1, R23.1, R25.1, SW1.1, SW2.1, U11.47 (VREG_PGND), U11.61 (GND), Y1.2 (G), Y1.4 (G)
- new net LED: Q7.1 (G), R25.2, U11.5 (GPIO3)
- new net RX_ADC_S: U11.40 (GPIO26/ADC0)
- new net RX_CMP_H: U11.36 (GPIO24)
- new net RX_CMP_L: U11.37 (GPIO25)
- new net RX_LEV_0: U11.32 (GPIO20)
- new net RX_LEV_1: U11.33 (GPIO21)
- new net RX_LEV_2: U11.34 (GPIO22)
- new net RX_LEV_3: U11.35 (GPIO23)
- new net SW: C22.2, R20.2, SW3.2, U11.2 (GPIO0)
- new net SWCLK: J3.1 (Pin_1), U11.24 (SWCLK)
- new net SWDIO: J3.3 (Pin_3), U11.25 (SWDIO)
- new net TX: Q6.1 (G), R23.2, U11.4 (GPIO2)
- new net TX_FET_N: U11.17 (GPIO13)
- new net TX_FET_P: U11.16 (GPIO12)
- new net TX_LEV_0: U11.14 (GPIO10)
- new net TX_LEV_1: U11.15 (GPIO11)
- new net XIN: R14.2, U11.21 (XIN)
- new net XOUT: R15.2, U11.22 (XOUT)
- new net usb/D+: R17.1
- new net usb/D-: R16.1
- new net ~{QSPI_SS}: R19.2, U11.60 (~{QSPI_SS})
- new net ~{RUN}: R13.2, U11.26 (RUN)
- no-connect marks 0 -> 22
Other:
- added sheet usb (usb.kicad_sch)
- note added: "Clock"
- note added: "Color LCSC# name isBaic wavelength Red C2286 KT-0603R o 620 Yellow C2289 xxxx o 589 White C2290 KT-0603W o --- Green C12624 KT-0603G x 525 Blue C2288 KT-0603B x 469 YGreen C2289 KT-0603YG x 576"
- note added: "Debug I/F"
- note added: "Input - Switch"
- note added: "Mechanical"
- note added: "Output - LED"
- note added: "Power"
- note added: "Red"
- note added: "USB Power"
- note added: "Yellow"
- note added: "for DVDD"
- note added: "for IOVDD"

Commit message: update sch
Other:
- added sheet spc500 (spc500.kicad_sch)

Commit message: update puns
Connections:
- net TX_LEV_0 is gone; now on net signal_N_H: U11.14 (GPIO10)
- net TX_LEV_1 is gone; now on net signal_N_L: U11.15 (GPIO11)
- net RX_LEV_0: no longer U11.32 (GPIO20)
- net RX_LEV_1: no longer U11.33 (GPIO21)
- net RX_LEV_2: no longer U11.34 (GPIO22)
- net RX_LEV_3: no longer U11.35 (GPIO23)
- net signal_L_H: now reaches U11.12 (GPIO8)
- net signal_L_L: now reaches U11.13 (GPIO9)
- net TX_FET_N: no longer names the net of U11.17 (GPIO13)
- net TX_FET_P: no longer names the net of U11.16 (GPIO12)
Changed lines of the file:
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@@
+	)
+	(no_connect
+		(at 187.96 83.82)
 	)
 	(no_connect
@@
 	)
 	(no_connect
-		(at 187.96 73.66)
-	)
-	(no_connect
 		(at 127 93.98)
 	)
@@
 	)
 	(no_connect
-		(at 187.96 71.12)
-	)
-	(no_connect
 		(at 187.96 86.36)
 	)
@@
 	)
 	(no_connect
+		(at 187.96 81.28)
+	)
+	(no_connect
 		(at 187.96 127)
 	)
-	(bus_entry
-		(at 200.66 106.68)
-		(size -2.54 2.54)
-		(stroke
-			(width 0)
-			(type default)
-		)
-	)
-	(bus_entry
-		(at 195.58 76.2)
-		(size -2.54 2.54)
-		(stroke
-			(width 0)
-			(type default)
-		)
-	)
-	(bus_entry
-		(at 200.66 99.06)
-		(size -2.54 2.54)
-		(stroke
-			(width 0)
-			(type default)
-		)
-	)
-	(bus_entry
-		(at 200.66 104.14)
-		(size -2.54 2.54)
-		(stroke
-			(width 0)
-			(type default)
-		)
-	)
-	(bus_entry
-		(at 195.58 73.66)
-		(size -2.54 2.54)
-		(stroke
-			(width 0)
-			(type default)
-		)
-	)
-	(bus_entry
-		(at 200.66 101.6)
-		(size -2.54 2.54)
-		(stroke
-			(width 0)
-			(type default)
-		)
-	)
 	(wire
 		(pts
@@
 	(wire
 		(pts
-			(xy 177.8 101.6) (xy 198.12 101.6)
-		)
-		(stroke
-			(width 0)
-			(type default)
-		)
-	)
-	(wire
-		(pts
 			(xy 97.79 25.4) (xy 95.25 25.4)
 		)
@@
 		)
 	)
-	(bus
-		(pts
-			(xy 200.66 46.99) (xy 200.66 106.68)
-		)
-		(stroke
-			(width 0)
-			(type default)
-		)
-	)
 	(wire
 		(pts
@@
 	(wire
 		(pts
+			(xy 177.8 76.2) (xy 187.96 76.2)
+		)
+		(stroke
+			(width 0)
+			(type default)
+		)
+	)
+	(wire
+		(pts
 			(xy 241.3 138.43) (xy 241.3 152.4)
 		)
@@
 		(pts
 			(xy 257.81 152.4) (xy 257.81 149.86)
+		)
+		(stroke
+			(width 0)
+			(type default)
+		)
+	)
+	(wire
+		(pts
+			(xy 177.8 73.66) (xy 187.96 73.66)
 		)
 		(stroke
@@
 	(wire
 		(pts
+			(xy 177.8 78.74) (xy 187.96 78.74)
+		)
+		(stroke
+			(width 0)
+			(type default)
+		)
+	)
+	(wire
+		(pts
 			(xy 187.96 93.98) (xy 177.8 93.98)
 		)
@@
 		)
 	)
-	(bus
-		(pts
-			(xy 215.9 46.99) (xy 200.66 46.99)
-		)
-		(stroke
-			(width 0)
-			(type default)
-		)
-	)
 	(wire
 		(pts
@@
 	(wire
 		(pts
-			(xy 187.96 73.66) (xy 177.8 73.66)
-		)
-		(stroke
-			(width 0)
-			(type default)
-		)
-	)
-	(wire
-		(pts
-			(xy 177.8 78.74) (xy 193.04 78.74)
-		)
-		(stroke
-			(width 0)
-			(type default)
-		)
-	)
-	(wire
-		(pts
 			(xy 187.96 58.42) (xy 177.8 58.42)
 		)
@@
 	(wire
 		(pts
-			(xy 177.8 106.68) (xy 198.12 106.68)
-		)
-		(stroke
-			(width 0)
-			(type default)
-		)
-	)
-	(wire
-		(pts
 			(xy 149.86 41.91) (xy 149.86 43.18)
 		)
@@
 	(wire
 		(pts
-			(xy 187.96 71.12) (xy 177.8 71.12)
+			(xy 177.8 71.12) (xy 187.96 71.12)
 		)
 		(stroke
@@
 		)
 	)
-	(bus
-		(pts
-			(xy 215.9 41.91) (xy 195.58 41.91)
-		)
-		(stroke
-			(width 0)
-			(type default)
-		)
-	)
-	(wire
-		(pts
-			(xy 177.8 109.22) (xy 198.12 109.22)
-		)
-		(stroke
-			(width 0)
-			(type default)
-		)
-	)
 	(wire
 		(pts
@@
 		)
 	)
-	(bus
-		(pts
-			(xy 195.58 41.91) (xy 195.58 76.2)
-		)
-		(stroke
-			(width 0)
-			(type default)
-		)
-	)
 	(wire
 		(pts
@@
 		(pts
 			(xy 88.9 53.34) (xy 88.9 50.8)
-		)
-		(stroke
-			(width 0)
-			(type default)
-		)
-	)
-	(wire
-		(pts
-			(xy 177.8 76.2) (xy 193.04 76.2)
-		)
-		(stroke
-			(width 0)
-			(type default)
-		)
-	)
-	(wire
-		(pts
-			(xy 177.8 104.14) (xy 198.12 104.14)
 		)
 		(stroke
@@
 		)
 	)
-	(label "signal_H_H"
+	(label "signal_L_H"
 		(at 215.9 71.12 0)
 		(effects
@@
 		)
 	)
-	(label "TX_LEV_0"
-		(at 187.96 76.2 180)
-		(effects
-			(font
-				(size 1.27 1.27)
-			)
-			(justify right bottom)
-		)
-	)
 	(label "XOUT"
 		(at 116.84 114.3 0)
@@
 		)
 	)
+	(label "signal_N_H"
+		(at 187.96 76.2 180)
+		(effects
+			(font
+				(size 1.27 1.27)
+			)
+			(justify right bottom)
+		)
+	)
 	(label "signal_N_L"
 		(at 215.9 81.28 0)
@@
 		)
 	)
-	(label "signal_H_L"
+	(label "signal_L_L"
 		(at 215.9 73.66 0)
 		(effects
@@
 		)
 	)
+	(label "signal_L_L"
+		(at 187.96 73.66 180)
+		(effects
+			(font
+				(size 1.27 1.27)
+			)
+			(justify right bottom)
+		)
+	)
 	(label "SPC500.L"
 		(at 279.4 71.12 180)
@@
 		)
 	)
-	(label "TX_LEV_[0..1]"
-		(at 215.9 41.91 180)
+	(label "signal_N_L"
+		(at 187.96 78.74 180)
 		(effects
 			(font
@@
 		)
 	)
-	(label "RX_LEV_[0..3]"
-		(at 215.9 46.99 180)
-		(effects
-			(font
-				(size 1.27 1.27)
-			)
-			(justify right bottom)
-		)
-	)
 	(label "RX_CMP_L"
 		(at 187.96 114.3 180)
@@
 		)
 	)
+	(label "signal_L_H"
+		(at 187.96 71.12 180)
+		(effects
+			(font
+				(size 1.27 1.27)
+			)
+			(justify right bottom)
+		)
+	)
 	(label "SWCLK"
 		(at 116.84 121.92 0)
@@
 		)
 	)
-	(label "TX_FET_N"
-		(at 187.96 83.82 180)
-		(effects
-			(font
-				(size 1.27 1.27)
-			)
-			(justify right bottom)
-		)
-	)
-	(label "TX_LEV_1"
-		(at 187.96 78.74 180)
-		(effects
-			(font
-				(size 1.27 1.27)
-			)
-			(justify right bottom)
-		)
-	)
-	(label "TX_FET_P"
-		(at 187.96 81.28 180)
-		(effects
-			(font
-				(size 1.27 1.27)
-			)
-			(justify right bottom)
-		)
-	)
